Commit message: update sim

File: nav/urdf/ranger_platform.xacro (robot description, xacro)
@@ -14,5 +14,5 @@
       </geometry>
       <material name="">
-        <color rgba="1 1 1 1"/>
+        <color rgba="0.6 0.6 0.6 1"/>
       </material>
     </visual>
@@ -25,5 +25,8 @@
     </collision>
   </link>
-<link name="fr_steering_wheel_link">
+  <gazebo reference="base_link">
+    <material>Gazebo/Grey</material>
+  </gazebo>
+  <link name="fr_steering_wheel_link">
     <inertial>
       <origin xyz="0.0001118 -0.0073218 -0.085228" rpy="0 0 0"/>
@@ -37,5 +40,5 @@
       </geometry>
       <material name="">
-        <color rgba="0 0 0 1"/>
+        <color rgba="0.3 0.3 0.3 1"/>
       </material>
     </visual>
@@ -47,4 +50,7 @@
     </collision>
   </link>
+  <gazebo reference="fr_steering_wheel_link">
+    <material>Gazebo/DarkGrey</material>
+  </gazebo>
   <link name="fr_wheel_link">
     <inertial>
@@ -59,5 +65,5 @@
       </geometry>
       <material name="">
-        <color rgba="1 1 1 1"/>
+        <color rgba="0.1 0.1 0.1 1"/>
       </material>
     </visual>
@@ -70,4 +76,7 @@
     </collision>
   </link>
+  <gazebo reference="fr_wheel_link">
+    <material>Gazebo/Black</material>
+  </gazebo>
   <link name="fl_steering_wheel_link">
     <inertial>
@@ -82,5 +91,5 @@
       </geometry>
       <material name="">
-        <color rgba="0 0 0 1"/>
+        <color rgba="0.3 0.3 0.3 1"/>
       </material>
     </visual>
@@ -92,4 +101,7 @@
     </collision>
   </link>
+  <gazebo reference="fl_steering_wheel_link">
+    <material>Gazebo/DarkGrey</material>
+  </gazebo>
   <link name="fl_wheel_link">
     <inertial>
@@ -104,5 +116,5 @@
       </geometry>
       <material name="">
-        <color rgba="1 1 1 1"/>
+        <color rgba="0.1 0.1 0.1 1"/>
       </material>
     </visual>
@@ -115,4 +127,7 @@
     </collision>
   </link>
+  <gazebo reference="fl_wheel_link">
+    <material>Gazebo/Black</material>
+  </gazebo>
   <link name="rl_steering_wheel_link">
     <inertial>
@@ -127,5 +142,5 @@
       </geometry>
       <material name="">
-        <color rgba="0 0 0 1"/>
+        <color rgba="0.3 0.3 0.3 1"/>
       </material>
     </visual>
@@ -137,4 +152,7 @@
     </collision>
   </link>
+  <gazebo reference="rl_steering_wheel_link">
+    <material>Gazebo/DarkGrey</material>
+  </gazebo>
   <link name="rl_wheel_link">
     <inertial>
@@ -149,5 +167,5 @@
       </geometry>
       <material name="">
-        <color rgba="1 1 1 1"/>
+        <color rgba="0.1 0.1 0.1 1"/>
       </material>
     </visual>
@@ -160,4 +178,7 @@
     </collision>
   </link>
+  <gazebo reference="rl_wheel_link">
+    <material>Gazebo/Black</material>
+  </gazebo>
   <link name="rr_steering_wheel_link">
     <inertial>
@@ -172,5 +193,5 @@
       </geometry>
       <material name="">
-        <color rgba="0 0 0 1"/>
+        <color rgba="0.3 0.3 0.3 1"/>
       </material>
     </visual>
@@ -182,4 +203,7 @@
     </collision>
   </link>
+  <gazebo reference="rr_steering_wheel_link">
+    <material>Gazebo/DarkGrey</material>
+  </gazebo>
   <link name="rr_wheel_link">
     <inertial>
@@ -194,5 +218,5 @@
       </geometry>
       <material name="">
-        <color rgba="1 1 1 1"/>
+        <color rgba="0.1 0.1 0.1 1"/>
       </material>
     </visual>
@@ -205,4 +229,7 @@
     </collision>
   </link>
+  <gazebo reference="rr_wheel_link">
+    <material>Gazebo/Black</material>
+  </gazebo>
   <joint name="fl_steering_wheel_joint" type="revolute">
     <origin xyz="0.445 0.28 0.0335" rpy="0 0 0"/>
